Commit message: Ignore commands for unattached servo' s. Identical to SSC32U

File: src/al5d_simulation/urdf/al5d.urdf (robot description, URDF)
Before this commit: robot lynxmotion_arm, 8 links, 7 joints
Joints:
- joint gripper_right2hand: mimic joint=gripper_left2hand multiplier=1 offset=0 -> (none)
